Commit message: Fix the localization bug which caused by non-centered (along x-axis) tf frame base_footprint

File: linorobot2/linorobot2_description/urdf/zbotlino_properties.urdf.xacro (robot description, xacro)
@@ -9,4 +9,6 @@
   <xacro:property name="wheel_pos_x" value="0.0" />
   <!-- <xacro:property name="wheel_pos_x" value="-0.13" /> -->
+  <!-- <xacro:property name="offset_x" value="0.0" /> -->
+  <xacro:property name="offset_x" value="0.13" />
   <!-- <xacro:property name="wheel_pos_y" value="0.14" /> -->
   <xacro:property name="wheel_pos_y" value="${base_width/2+wheel_width/2}" />
@@ -17,8 +19,8 @@
   <xacro:property name="rear_caster_wheel" value="false" />
   <xacro:property name="laser_pose">
-    <origin xyz="0.12 0 0.07" rpy="0 0 0"/>
+    <origin xyz="${0.12+offset_x} 0 0.07" rpy="0 0 0"/>
   </xacro:property>
   <xacro:property name="depth_sensor_pose">
-    <origin xyz="0.2 0.0 0.045" rpy="0 0 0"/>
+    <origin xyz="${0.2+offset_x} 0.0 0.045" rpy="0 0 0"/>
   </xacro:property>
 </robot>

Commit message: Update zbotlino_properties.urdf.xacro. More accurate.

File: linorobot2/linorobot2_description/urdf/zbotlino_properties.urdf.xacro (robot description, xacro)
@@ -1,5 +1,5 @@
 <?xml version="1.0"?>
 <robot xmlns:xacro="http://ros.org/wiki/xacro">
-  <xacro:property name="base_length" value="0.376" />
+  <xacro:property name="base_length" value="0.3757" />
   <xacro:property name="base_width" value="0.28" />
   <xacro:property name="base_height" value="0.003" />
@@ -10,8 +10,9 @@
   <!-- <xacro:property name="wheel_pos_x" value="-0.13" /> -->
   <!-- <xacro:property name="offset_x" value="0.0" /> -->
-  <xacro:property name="offset_x" value="0.13" />
+  <xacro:property name="offset_x" value="${base_length/2-0.055}" />
   <!-- <xacro:property name="wheel_pos_y" value="0.14" /> -->
-  <xacro:property name="wheel_pos_y" value="${base_width/2+wheel_width/2}" />
-  <xacro:property name="wheel_pos_z" value="-0.06" />
+  <xacro:property name="wheel_pos_y" value="${base_width/2+wheel_width/2+0.01}" />
+  <!--<xacro:property name="wheel_pos_z" value="-0.06" />-->
+  <xacro:property name="wheel_pos_z" value="${-wheel_radius+0.0005}" />
   <xacro:property name="wheel_mass" value=".1" />
   <xacro:property name="wheel_torque" value="20" />
@@ -19,5 +20,6 @@
   <xacro:property name="rear_caster_wheel" value="false" />
   <xacro:property name="laser_pose">
-    <origin xyz="${0.12+offset_x} 0 0.07" rpy="0 0 0"/>
+    <!--<origin xyz="${0.12+offset_x} 0 0.07" rpy="0 0 0"/>-->
+    <origin xyz="${base_length/2+offset_x-0.085} 0 0.088" rpy="0 0 0"/>
   </xacro:property>
   <xacro:property name="depth_sensor_pose">

Commit message: use humble's default nav2_params as navigation.yaml

File: linorobot2/linorobot2_description/urdf/zbotlino_properties.urdf.xacro (robot description, xacro)
@@ -2,4 +2,5 @@
 <robot xmlns:xacro="http://ros.org/wiki/xacro">
   <xacro:property name="base_length" value="0.3757" />
+  <!-- <xacro:property name="base_length" value="0.6" /> -->
   <xacro:property name="base_width" value="0.28" />
   <xacro:property name="base_height" value="0.003" />

Commit message: Fine tune zbotlino_properties.urdf.xacro & navigation.yaml to see the footprint influence.

File: linorobot2/linorobot2_description/urdf/zbotlino_properties.urdf.xacro (robot description, xacro)
@@ -1,6 +1,6 @@
 <?xml version="1.0"?>
 <robot xmlns:xacro="http://ros.org/wiki/xacro">
-  <xacro:property name="base_length" value="0.3757" />
-  <!-- <xacro:property name="base_length" value="0.6" /> -->
+  <!-- <xacro:property name="base_length" value="0.3757" /> -->
+  <xacro:property name="base_length" value="0.55" />
   <xacro:property name="base_width" value="0.28" />
   <xacro:property name="base_height" value="0.003" />

Commit message: Update zbotlino_properties.urdf.xacro. Add more laser properties.

File: linorobot2/linorobot2_description/urdf/zbotlino_properties.urdf.xacro (robot description, xacro)
@@ -21,8 +21,11 @@
   <xacro:property name="rear_caster_wheel" value="false" />
   <xacro:property name="laser_pose">
-    <!--<origin xyz="${0.12+offset_x} 0 0.07" rpy="0 0 0"/>-->
+    <!-- zbot lino 1.5 rplidar -->
     <origin xyz="${base_length/2+offset_x-0.085} 0 0.088" rpy="0 0 0"/>
   </xacro:property>
-  <xacro:property name="laser_pose1">
+  <xacro:property name="laser_pose_nanoscan3_front">
+    <origin xyz="${base_length/2+offset_x-0.06} 0 0.14" rpy="0 0 0"/>
+  </xacro:property>
+  <xacro:property name="laser_pose_front_inverted">
     <origin xyz="${base_length/2+offset_x} 0 0.088" rpy="3.1415 0 0"/>
   </xacro:property>
