Commit message: Add zbotlinolong related files. This is for simulation.

File: linorobot2/linorobot2_description/urdf/zbotlinolong_properties.urdf.xacro (robot description, xacro)
@@ -1,5 +1,5 @@
 <?xml version="1.0"?>
 <robot xmlns:xacro="http://ros.org/wiki/xacro">
-  <xacro:property name="base_length" value="0.3757" />
+  <xacro:property name="base_length" value="0.55" />
   <xacro:property name="base_width" value="0.28" />
   <xacro:property name="base_height" value="0.003" />
