Commit message: Fix typo

File: linorobot2/linorobot2_description/urdf/zbotlino2_properties.urdf.xacro (robot description, xacro)
@@ -36,14 +36,14 @@
   <xacro:property name="sonic_offset_z" value="0.05" />
   <xacro:property name="range1_sensor_pose">
-    <origin xyz="${offset_x+sonic_offset_x} ${sonic_offset_y} ${-base_height/2-sonic_offic_z}" rpy="0 0 0"/>
+    <origin xyz="${offset_x+sonic_offset_x} ${sonic_offset_y} ${-base_height/2-sonic_offset_z}" rpy="0 0 0"/>
   </xacro:property>
   <xacro:property name="range2_sensor_pose">
-    <origin xyz="${offset_x+sonic_offset_x} ${-sonic_offset_y} ${-base_height/2-sonic_offic_z}" rpy="0 0 0"/>
+    <origin xyz="${offset_x+sonic_offset_x} ${-sonic_offset_y} ${-base_height/2-sonic_offset_z}" rpy="0 0 0"/>
   </xacro:property>
   <xacro:property name="range3_sensor_pose">
-    <origin xyz="${offset_x-sonic_offset_x} ${-sonic_offset_y} ${-base_height/2-sonic_offic_z}" rpy="0 0 3.1415"/>
+    <origin xyz="${offset_x-sonic_offset_x} ${-sonic_offset_y} ${-base_height/2-sonic_offset_z}" rpy="0 0 3.1415"/>
   </xacro:property>
   <xacro:property name="range4_sensor_pose">
-    <origin xyz="${offset_x-sonic_offset_x} ${sonic_offset_y} ${-base_height/2-sonic_offic_z}" rpy="0 0 3.1415"/>
+    <origin xyz="${offset_x-sonic_offset_x} ${sonic_offset_y} ${-base_height/2-sonic_offset_z}" rpy="0 0 3.1415"/>
   </xacro:property>
 </robot>

Commit message: 1. Add tf remappings in description.launch.py for namepsace support 2. Add zbotlino2a. Replace front depth_sensor with rear camera 3. Modify navigation.launch.py to allow rviz_config 4. Modify zbotlino2's navigation.yaml. Speed up.

File: linorobot2/linorobot2_description/urdf/zbotlino2_properties.urdf.xacro (robot description, xacro)
@@ -32,4 +32,8 @@
     <origin xyz="${0.2+offset_x} 0.0 0.045" rpy="0 0 0"/>
   </xacro:property>
+  <xacro:property name="camera_rear">
+    <origin xyz="${offset_x-0.3} 0.0 0.045" rpy="0 0 3.14159"/>
+    <!-- <origin xyz="${offset_x-0.3} 0.0 0.045" rpy="0 3.14159 0"/> -->
+  </xacro:property>
   <xacro:property name="sonic_offset_x" value="0.38" />
   <xacro:property name="sonic_offset_y" value="0.162" />

Commit message: change zbotlino2_properties  - property camera_rear: offset from 0.3 to 0.35

File: linorobot2/linorobot2_description/urdf/zbotlino2_properties.urdf.xacro (robot description, xacro)
@@ -33,5 +33,5 @@
   </xacro:property>
   <xacro:property name="camera_rear">
-    <origin xyz="${offset_x-0.3} 0.0 0.045" rpy="0 0 3.14159"/>
+    <origin xyz="${offset_x-0.35} 0.0 0.045" rpy="0 0 3.14159"/>
     <!-- <origin xyz="${offset_x-0.3} 0.0 0.045" rpy="0 3.14159 0"/> -->
   </xacro:property>
