Commit message: 1. Modify zbotlino_properties.urdf.xacro to add new laser properties laser_pose1 for inverted case 2. Clarify a serious problem. plugins in local_costmap should be [voxel_layer, inflatiolayer]    instead of [obstacle_layer, inflation_layer] 3. Add footprint definition in navigation.yaml 4. User navigation.yaml in navigation.launch.py

File: linorobot2/linorobot2_description/urdf/robots/zbotlino.urdf.xacro (robot description, xacro)
@@ -56,5 +56,6 @@
   <xacro:imu/>
   <xacro:generic_laser>
-    <xacro:insert_block name="laser_pose" />
+    <!-- <xacro:insert_block name="laser_pose" /> -->
+    <xacro:insert_block name="laser_pose1" />
   </xacro:generic_laser>
   <xacro:depth_sensor>

File: linorobot2/linorobot2_description/urdf/zbotlino_properties.urdf.xacro (robot description, xacro)
@@ -23,4 +23,7 @@
     <origin xyz="${base_length/2+offset_x-0.085} 0 0.088" rpy="0 0 0"/>
   </xacro:property>
+  <xacro:property name="laser_pose1">
+    <origin xyz="${base_length/2+offset_x} 0 0.088" rpy="3.1415 0 0"/>
+  </xacro:property>
   <xacro:property name="depth_sensor_pose">
     <origin xyz="${0.2+offset_x} 0.0 0.045" rpy="0 0 0"/>

Commit message: change zbotlino.urdf.xacro & zbotlino_properties.urdf.xacro back to real zbot lino v1.5

File: linorobot2/linorobot2_description/urdf/robots/zbotlino.urdf.xacro (robot description, xacro)
@@ -56,6 +56,6 @@
   <xacro:imu/>
   <xacro:generic_laser>
-    <!-- <xacro:insert_block name="laser_pose" /> -->
-    <xacro:insert_block name="laser_pose1" />
+    <xacro:insert_block name="laser_pose" />
+    <!-- <xacro:insert_block name="laser_pose1" /> -->
   </xacro:generic_laser>
   <xacro:depth_sensor>

File: linorobot2/linorobot2_description/urdf/zbotlino_properties.urdf.xacro (robot description, xacro)
@@ -1,6 +1,6 @@
 <?xml version="1.0"?>
 <robot xmlns:xacro="http://ros.org/wiki/xacro">
-  <!-- <xacro:property name="base_length" value="0.3757" /> -->
-  <xacro:property name="base_length" value="0.55" />
+  <xacro:property name="base_length" value="0.3757" />
+  <!-- <xacro:property name="base_length" value="0.55" /> -->
   <xacro:property name="base_width" value="0.28" />
   <xacro:property name="base_height" value="0.003" />
