Commit message: Add zbotlinosick1.urdf.xacro & zbotlinoinvert.urdf.xacro

File: linorobot2/linorobot2_description/urdf/robots/zbotlinoinvert.urdf.xacro (robot description, xacro)
@@ -56,5 +56,5 @@
   <xacro:imu/>
   <xacro:generic_laser>
-    <xacro:insert_block name="laser_pose" />
+    <xacro:insert_block name="laser_pose_front_inverted" />
   </xacro:generic_laser>
   <xacro:depth_sensor>

File: linorobot2/linorobot2_description/urdf/robots/zbotlinosick1.urdf.xacro (robot description, xacro)
@@ -56,5 +56,5 @@
   <xacro:imu/>
   <xacro:generic_laser>
-    <xacro:insert_block name="laser_pose" />
+    <xacro:insert_block name="laser_pose_nanoscan3_front" />
   </xacro:generic_laser>
   <xacro:depth_sensor>

File: linorobot2/linorobot2_description/urdf/zbotlino_properties.urdf.xacro (robot description, xacro)
@@ -21,8 +21,10 @@
   <xacro:property name="rear_caster_wheel" value="false" />
   <xacro:property name="laser_pose">
-    <!--<origin xyz="${0.12+offset_x} 0 0.07" rpy="0 0 0"/>-->
     <origin xyz="${base_length/2+offset_x-0.085} 0 0.088" rpy="0 0 0"/>
   </xacro:property>
-  <xacro:property name="laser_pose1">
+  <xacro:property name="laser_pose_nanoscan3_front">
+    <origin xyz="${base_length/2+offset_x-0.06} 0 0.14" rpy="0 0 0"/>
+  </xacro:property>
+  <xacro:property name="laser_pose_front_inverted">
     <origin xyz="${base_length/2+offset_x} 0 0.088" rpy="3.1415 0 0"/>
   </xacro:property>
