Commit message: Add range_sensor tf trees

File: linorobot2/linorobot2_description/urdf/robots/zbotlinosick1.urdf.xacro (robot description, xacro)
@@ -9,4 +9,6 @@
   <xacro:include filename="$(find linorobot2_description)/urdf/sensors/generic_laser.urdf.xacro" />
   <xacro:include filename="$(find linorobot2_description)/urdf/sensors/depth_sensor.urdf.xacro" />
+  <xacro:include filename="$(find linorobot2_description)/urdf/sensors/ultrasonic.urdf.xacro" />
+  <xacro:include filename="$(find linorobot2_description)/urdf/sensors/generic_ultrasonic.urdf.xacro" />
   <xacro:include filename="$(find linorobot2_description)/urdf/controllers/diff_drive.urdf.xacro" />
   <xacro:base
@@ -61,4 +63,10 @@
     <xacro:insert_block name="depth_sensor_pose" />
   </xacro:depth_sensor>
+  <xacro:range1>
+    <xacro:insert_block name="range1_sensor_pose" />
+  </xacro:range1>
+  <xacro:range2>
+    <xacro:insert_block name="range2_sensor_pose" />
+  </xacro:range2>
   <xacro:diff_drive_controller
     wheel_separation="${wheel_pos_y * 2}"

File: linorobot2/linorobot2_description/urdf/zbotlino_properties.urdf.xacro (robot description, xacro)
@@ -28,3 +28,9 @@
     <origin xyz="${0.2+offset_x} 0.0 0.045" rpy="0 0 0"/>
   </xacro:property>
+  <xacro:property name="range1_sensor_pose">
+    <origin xyz="${offset_x+base_length/2-0.02/2} 0.0 ${-base_height/2-0.01/2}" rpy="0 0 0"/>
+  </xacro:property>
+  <xacro:property name="range2_sensor_pose">
+    <origin xyz="${-0.055+0.02/2} 0.0 ${-base_height/2-0.01/2}" rpy="0 0 3.1415"/>
+  </xacro:property>
 </robot>
