Commit message: Update zbotlin2.urdf.xacro & zbtolino2_properties.urdf.xacro for four ultrasonic sensors.

File: linorobot2/linorobot2_description/urdf/robots/zbotlino2.urdf.xacro (robot description, xacro)
@@ -72,4 +72,10 @@
     <xacro:insert_block name="range2_sensor_pose" />
   </xacro:range2>
+  <xacro:range3>
+    <xacro:insert_block name="range3_sensor_pose" />
+  </xacro:range3>
+  <xacro:range4>
+    <xacro:insert_block name="range4_sensor_pose" />
+  </xacro:range4>
   <xacro:diff_drive_controller
     wheel_separation="${wheel_pos_y * 2}"

File: linorobot2/linorobot2_description/urdf/zbotlino2_properties.urdf.xacro (robot description, xacro)
@@ -32,9 +32,18 @@
     <origin xyz="${0.2+offset_x} 0.0 0.045" rpy="0 0 0"/>
   </xacro:property>
+  <xacro:property name="sonic_offset_x" value="0.38" />
+  <xacro:property name="sonic_offset_y" value="0.162" />
+  <xacro:property name="sonic_offset_z" value="0.05" />
   <xacro:property name="range1_sensor_pose">
-    <origin xyz="${offset_x+base_length/2-0.02/2} 0.0 ${-base_height/2-0.01/2}" rpy="0 0 0"/>
+    <origin xyz="${offset_x+sonic_offset_x} ${sonic_offset_y} ${-base_height/2-sonic_offic_z}" rpy="0 0 0"/>
   </xacro:property>
   <xacro:property name="range2_sensor_pose">
-    <origin xyz="${-0.055+0.02/2} 0.0 ${-base_height/2-0.01/2}" rpy="0 0 3.1415"/>
+    <origin xyz="${offset_x+sonic_offset_x} ${-sonic_offset_y} ${-base_height/2-sonic_offic_z}" rpy="0 0 0"/>
+  </xacro:property>
+  <xacro:property name="range3_sensor_pose">
+    <origin xyz="${offset_x-sonic_offset_x} ${-sonic_offset_y} ${-base_height/2-sonic_offic_z}" rpy="0 0 3.1415"/>
+  </xacro:property>
+  <xacro:property name="range4_sensor_pose">
+    <origin xyz="${offset_x-sonic_offset_x} ${sonic_offset_y} ${-base_height/2-sonic_offic_z}" rpy="0 0 3.1415"/>
   </xacro:property>
 </robot>
