Commit message: Update xacro for two lidars

File: linorobot2/linorobot2_description/urdf/sensors/generic_laser.urdf.xacro (robot description, xacro)
@@ -2,4 +2,33 @@
 <robot xmlns:xacro="http://ros.org/wiki/xacro">
   <xacro:include filename="$(find linorobot2_description)/urdf/sensors/laser.urdf.xacro" />
+  <xacro:macro name="laser1" params="*origin">
+    <xacro:laser
+      update_rate="10"
+      ray_count="270"
+      min_angle="-2.3562"
+      max_angle="2.3562"
+      min_range="0.08"
+      max_range="40.0"
+      frame_id="laser1"
+      topic_name="scan1"
+    >
+      <xacro:insert_block name="origin" />
+    </xacro:laser>
+  </xacro:macro>
+  <xacro:macro name="laser2" params="*origin">
+    <xacro:laser
+      update_rate="10"
+      ray_count="270"
+      min_angle="-2.3562"
+      max_angle="2.3562"
+      min_range="0.08"
+      max_range="40.0"
+      frame_id="laser2"
+      topic_name="scan2"
+    >
+      <xacro:insert_block name="origin" />
+    </xacro:laser>
+  </xacro:macro>
+  <!--  -->
   <xacro:macro name="generic_laser" params="*origin">
     <xacro:laser

File: linorobot2/linorobot2_description/urdf/zbotlino_properties.urdf.xacro (robot description, xacro)
@@ -22,4 +22,7 @@
     <origin xyz="${base_length/2+offset_x-0.06} 0 0.14" rpy="0 0 0"/>
   </xacro:property>
+  <xacro:property name="laser_pose_nanoscan3_back">
+    <origin xyz="${0.05-0.055} 0 0.14" rpy="0 0 3.1415"/>
+  </xacro:property>
   <xacro:property name="laser_pose_front_inverted">
     <origin xyz="${base_length/2+offset_x} 0 0.088" rpy="3.1415 0 0"/>
